File: template.brd (EAGLE design)
At the start: 25.4 x 32.4 mm, 5 parts

Commit message: Renamed GPIO4 & GPIO5 as SDA and SCL respectively to suit their default i2c states.
Connections:
- net GPIO4 renamed SDA
- net GPIO5 renamed SCL
Changed lines of the file:
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@@
 <contactref element="IC1" pad="19"/>
 </signal>
-<signal name="GPIO4">
+<signal name="SDA">
 <contactref element="IC1" pad="21"/>
 </signal>
@@
 <contactref element="IC1" pad="24"/>
 </signal>
-<signal name="GPIO5">
+<signal name="SCL">
 <contactref element="IC1" pad="22"/>
 </signal>
